File: tests/fixtures/despertador-routed/despertador_inteligente.kicad_sch (KiCad schematic)
At the start: 24 parts, among them J1 Conector ICSP, J2 CSE, U1 ATtiny85-20S, U2 MPU-6050, U3 MAX30102, U4 RFM69CW

Commit message: post-D3 contecto actualizado CONTEXT-V3.md y frecciones D3 en ocs/dogfooding/dogfood3-fricciones.md
Parts:
- removed TP6: TestPoint, TestPoint:TestPoint_Pad_D2.0mm, symbol Connector:TestPoint
- J1: now left out of the parts list
Connections:
- net MOSI: now also R3.2, U1.1 (~{RESET}/PB5); no longer U1.5 (AREF/PB0), U4.5 (NSS)
- net INT_SENS renamed SCL
- net SCL: no longer R3.2, U2.12 (INT), U3.13 (~{INT})
- net RESET: no longer names the net of J1.5
- net RESET: no longer U1.1 (~{RESET}/PB5)
- new net NSS: U1.5 (AREF/PB0), U4.5 (NSS)
- no-connect marks 15 -> 16
